File: hardware/electronics/motion_controller/motion_controller.kicad_pcb (KiCad board)
At the start: 2 copper layers, 181 parts, among them K1 CONN_3, K10 CONN_3, K11 CONN_3, K12 CONN_3, K13 CONN_3, K14 CONN_3, K15 CONN_3, K2 CONN_3, K3 CONN_3, K4 CONN_3, K5 CONN_3, K6 CONN_3, K7 CONN_3, K8 CONN_3, K9 CONN_3, P1 CONN_2, P10 CONN_4, P11 CONN_4, P12 CONN_4, P13 CONN_2, P14 CONN_2, P15 CONN_2, P16 CONN_2, P17 CONN_2, P18 CONN_2, P19 CONN_2X2, P2 CONN_5X2, P20 CONN_2X2, P21 CONN_2, P22 CONN_2, P23 CONN_2, P24 CONN_2, P25 CONN_2, P26 CONN_2X2, P27 CONN_2, P28 CONN_2, P29 CONN_2, P3 CONN_2X2, P4 CONN_2, P5 CONN_34X2, P6 CONN_4, P7 CONN_4, P8 CONN_4, P9 CONN_4, U1 TEENSY3.1, U10 OP07, U11 OP07, U12 OP07, U13 OP07, U14 OP07, U15 OP07, U16 OP07, U17 MEA1D0512SC, U2 NC7WZ04, U3 NC7WZ16, U4 NC7WZ16, U5 SSR_DC_6PIN, U6 MAX6176AASA+, U7 OP07, U8 OP07, U9 OP07

Commit message: Worked on motion controller PCB layout.
Parts:
- moved R54 739.0 mm to (718.7, -70.2)
- moved U16 727.1 mm to (731.1, -70.4)
- moved R44 724.8 mm to (699.4, -77.2)
- moved R45 721.2 mm to (688.2, -77.4)
- moved U15 719.6 mm to (700.1, -70.8)
- moved C21 718.9 mm to (718.4, -83.2)
- moved R46 716.8 mm to (688.1, -74.2)
- moved R64 697.9 mm to (688.7, -64.1)
- moved C20 697.2 mm to (718.2, -86.4)
- moved R65 694.2 mm to (718.9, -63.6)
- moved C18 693.0 mm to (687.5, -84.5)
- moved R85 692.1 mm to (738.9, -63.6)
- moved D10 691.4 mm to (738.8, -70.7)
- moved R84 689.0 mm to (738.9, -66.4)
- moved C19 688.9 mm to (687.5, -81.8)
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
Commit message: Worked on layout of analog input subsystem.
Parts:
- moved R85 492.3 mm to (273.3, 96.3), turned to 270 degrees
- moved R84 491.6 mm to (273.3, 91.2), turned to 270 degrees
- moved D10 487.6 mm to (280.4, 95.8)
- moved U16 479.4 mm to (277.1, 83.6), turned to 180 degrees
- moved R83 475.9 mm to (259.3, 96.3), turned to 270 degrees
- moved R50 475.8 mm to (283.0, 83.6), turned to 270 degrees
- moved R82 475.3 mm to (259.3, 91.2), turned to 270 degrees
- moved C20 474.8 mm to (277.9, 91.2), turned to 270 degrees
- moved K15 473.6 mm to (278.1, 54.6)
- moved C21 473.1 mm to (273.3, 77.0), turned to 90 degrees
- moved D9 471.5 mm to (266.4, 95.8)
- moved R54 467.4 mm to (273.3, 71.6), turned to 90 degrees
- moved R52 466.9 mm to (273.3, 66.5), turned to 270 degrees
- moved R51 464.3 mm to (277.1, 66.5), turned to 270 degrees
- moved U15 463.4 mm to (263.1, 83.6), turned to 180 degrees
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Connections:
- C1 pad 2: /GND -> /AGND
- C10 pad 2: /GND -> /AGND
- C11 pad 2: /GND -> /AGND
- C12 pad 2: /GND -> /AGND
- C13 pad 2: /GND -> /AGND
- C14 pad 2: /GND -> /AGND
- C16 pad 2: /GND -> /AGND
- C17 pad 2: /GND -> /AGND
- C18 pad 2: /GND -> /AGND
- C19 pad 2: /GND -> /AGND
- C2 pad 2: /GND -> /AGND
- C20 pad 2: /GND -> /AGND
- C21 pad 2: /GND -> /AGND
- C3 pad 2: /GND -> /AGND
- C4 pad 2: /GND -> /AGND
- C5 pad 2: /GND -> /AGND
- C6 pad 2: /GND -> /AGND
- C7 pad 2: /GND -> /AGND
- C8 pad 2: /GND -> /AGND
- C9 pad 2: /GND -> /AGND
- R56 pad 1: /GND -> /AGND
- R57 pad 1: /GND -> /AGND
- R58 pad 1: /GND -> /AGND
- R59 pad 1: /GND -> /AGND
- R60 pad 1: /GND -> /AGND
- R61 pad 1: /GND -> /AGND
- R62 pad 1: /GND -> /AGND
- R63 pad 1: /GND -> /AGND
- R64 pad 1: /GND -> /AGND
- R65 pad 1: /GND -> /AGND

Commit message: Added PJRC SD card. Changed so that double schottky diodes in a analog clamp use AGND instead of GND. Worked on layout.
Parts:
- added U18: PJRC_SD_CARD, PJRC_SD_CARD, F.Cu at (58.4, 113.0)
- moved U17 524.8 mm to (124.5, 83.8), turned to 270 degrees
- moved C25 522.4 mm to (130.2, 78.7), turned to 270 degrees
- moved U4 484.6 mm to (116.1, 8.64)
- moved C23 484.6 mm to (122.6, 7.11)
- moved P28 484.6 mm to (114.7, -2.54)
- moved P29 484.6 mm to (126.6, -2.67)
- moved P21 470.2 mm to (46.2, -0.51)
- moved P22 470.2 mm to (59.7, 0.00)
- moved U3 470.2 mm to (52.7, 9.91)
- moved C22 470.2 mm to (58.2, 9.14)
- moved C15 462.1 mm to (227.8, -14.4)
- moved P20 462.1 mm to (218.7, -18.2)
- moved P19 462.1 mm to (210.3, -18.4)
- moved U2 462.1 mm to (227.1, -18.8)
- moved P23 431.0 mm to (70.2, 131.4)
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Connections:
- D1 pad 1: /GND -> /AGND
- D10 pad 1: /GND -> /AGND
- D2 pad 1: /GND -> /AGND
- D3 pad 1: /GND -> /AGND
- D4 pad 1: /GND -> /AGND
- D5 pad 1: /GND -> /AGND
- D6 pad 1: /GND -> /AGND
- D7 pad 1: /GND -> /AGND
- D8 pad 1: /GND -> /AGND
- D9 pad 1: /GND -> /AGND

Commit message: Finished initial layout of motion controller pcb.
Parts:
- added P30: CONN_1, MOUNT_HOLE_4_40, F.Cu at (54.6, 54.6)
- added P31: CONN_1, MOUNT_HOLE_4_40, F.Cu at (313.7, 54.6)
- added P32: CONN_1, MOUNT_HOLE_4_40, F.Cu at (313.7, 142.2)
- added P33: CONN_1, MOUNT_HOLE_4_40, F.Cu at (54.6, 142.2)
- moved P20 164.4 mm to (295.9, 127.0)
- moved P19 160.5 mm to (278.1, 127.0)
- moved C15 145.7 mm to (285.8, 119.4), turned to 180 degrees
- moved U2 145.5 mm to (285.8, 114.3), turned to 180 degrees
- moved C22 77.9 mm to (105.4, 71.1)
- moved P21 75.3 mm to (97.8, 54.4)
- moved U3 74.3 mm to (102.9, 64.8), turned to 180 degrees
- moved P22 72.7 mm to (108.0, 54.4)
- moved C24 66.7 mm to (139.1, 104.8)
- moved U6 66.7 mm to (142.2, 111.8)
- moved C23 64.4 mm to (129.5, 71.1)
- moved P28 57.4 mm to (121.9, 54.4)
- moved P29 57.3 mm to (132.1, 54.4)
- moved U4 57.2 mm to (127.0, 64.8), turned to 180 degrees
- moved P2 38.6 mm to (77.5, 55.9), turned to 0 degrees
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Other:
- board outline added: 266.7 x 95.3 mm
- net class Power added: clearance 0.254, trace_width 0.508, via_dia 0.889, via_drill 0.635

Commit message: Finished preliminary routing of motion controller PCB.
Parts:
- moved K2 97.8 mm to (66.0, 141.2)
- moved K4 97.8 mm to (76.2, 141.2)
- moved K1 97.8 mm to (61.0, 141.2)
- moved K3 97.8 mm to (71.1, 141.2)
- moved K5 97.8 mm to (81.3, 141.2)
- moved P27 47.0 mm to (50.8, 121.9)
- moved U18 45.7 mm to (58.4, 73.7)
- moved P26 45.5 mm to (76.2, 120.7)
- moved P3 45.5 mm to (85.1, 120.7)
- moved C15 32.6 mm to (253.2, 116.6), turned to 90 degrees
- moved R27 28.1 mm to (124.5, 132.1)
- moved P13 27.9 mm to (127.0, 142.5)
- moved P14 27.9 mm to (137.2, 142.5)
- moved P15 27.9 mm to (147.3, 142.5)
- moved P16 27.9 mm to (157.5, 142.5)
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Connections:
- K1 pad 2: /5V_SEL -> /5V_EXT
- K2 pad 2: /5V_SEL -> /5V_EXT
- K3 pad 2: /5V_SEL -> /5V_EXT
- K4 pad 2: /5V_SEL -> /5V_EXT
- K5 pad 2: /5V_SEL -> /5V_EXT
Routing:
- net /AGND: track 0.00 -> 835.1 mm
- net /GND: track 0.00 -> 791.2 mm
- net /3V3_TNY: track 0.00 -> 317.1 mm, vias 0 -> 6
- net /+12V: track 0.00 -> 309.9 mm
- net /DIR0: track 0.00 -> 289.7 mm
- net /HW_EN: track 0.00 -> 276.6 mm, vias 0 -> 2
- net /CLK1: track 0.00 -> 249.6 mm
- net /CLK0: track 0.00 -> 239.4 mm
- net /-12V: track 0.00 -> 233.1 mm, vias 0 -> 1
- net /5V_SEL: track 0.00 -> 232.1 mm
- net /DIR4: track 0.00 -> 230.1 mm
- net /SG9: track 0.00 -> 227.9 mm
- net /CLK4: track 0.00 -> 225.8 mm
- net /DIR1: track 0.00 -> 219.1 mm
- net /5V_TNY: track 0.00 -> 209.6 mm
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Other:
- net class Power: trace_width 0.508 -> 0.381

Commit message: Worked on motion controller PCB annotation, routing and layout.
Parts:
- U1: value TEENSY3.1 -> TEENSY3.X
- moved P3 47.1 mm to (87.6, 73.7)
- moved C25 13.3 mm to (116.8, 82.5)
- moved C15 8.84 mm to (261.6, 119.4)
- moved P20 7.95 mm to (293.6, 119.9)
- moved U2 7.64 mm to (266.7, 119.4)
- moved P4 7.23 mm to (299.7, 104.1), turned to 90 degrees
- moved P19 7.15 mm to (278.9, 119.9)
- moved R27 5.24 mm to (121.2, 128.0)
- moved P26 5.08 mm to (81.3, 120.7)
- moved U3 5.08 mm to (102.9, 69.8), turned to 0 degrees
- moved U4 5.08 mm to (127.0, 69.8), turned to 0 degrees
- moved C23 2.84 mm to (132.1, 69.8), turned to 270 degrees
- moved C22 2.84 mm to (108.0, 69.8), turned to 270 degrees
Routing:
- net /AGND: track 835.1 -> 0.00 mm
- net /GND: track 791.2 -> 50.6 mm
- net /3V3_TNY: track 317.1 -> 0.00 mm, vias 6 -> 0
- net /+12V: track 309.9 -> 0.00 mm
- net /DIR0: track 289.7 -> 0.00 mm
- net /HW_EN: track 276.6 -> 0.00 mm, vias 2 -> 0
- net /CLK1: track 249.6 -> 0.00 mm
- net /CLK0: track 239.4 -> 0.00 mm
- net /-12V: track 233.1 -> 0.00 mm, vias 1 -> 0
- net /5V_SEL: track 232.1 -> 0.00 mm
- net /DIR4: track 230.1 -> 0.00 mm
- net /SG9: track 227.9 -> 0.00 mm
- net /CLK4: track 225.8 -> 0.00 mm
- net /DIR1: track 219.1 -> 0.00 mm
- net /5V_TNY: track 209.6 -> 0.00 mm
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Other:
- net class Default: trace_width 0.254 -> 0.381
- board text added: "CLK0"
- board text added: "CLK1"
- board text added: "CLK2"
- board text added: "DIR0"
- board text added: "DIR1"
- board text added: "DIR2"
- board text added: "ENABLE"
- board text added: "F/T SENSOR"
- board text added: "GND"
- board text added: "MOTOR 0"
- board text added: "MOTOR 1"
- board text added: "MOTOR 2"
- board text added: "SG0"
- board text added: "SG1"
- board text added: "SG2"
- board text added: "SG3"
- board text added: "SG4"
- board text added: "SG5"
- board text added: "SG6"
- board text added: "SG7"
- board text added: "SG8"
- board text added: "SG9"
- board text added: "V+"
- board text added: "V-"

Commit message: Finished motion controller pcb annotation and re-routed board.
Parts:
- moved P4 208.8 mm to (91.4, 118.6)
- moved P20 6.83 mm to (298.2, 114.8), turned to 180 degrees
- moved P19 6.51 mm to (283.0, 114.8), turned to 180 degrees
- moved C15 5.11 mm to (263.9, 114.8)
- moved U2 5.11 mm to (269.0, 114.8)
- moved R27 3.88 mm to (124.5, 126.0)
- moved P27 3.05 mm to (50.8, 118.9)
- moved P26 2.17 mm to (80.5, 118.6)
- moved R47 1.85 mm to (98.6, 126.5)
- moved U5 1.85 mm to (107.2, 118.9)
- moved C22 1.52 mm to (108.0, 71.4)
- moved C23 1.52 mm to (132.1, 71.4)
- moved U3 1.52 mm to (102.9, 71.4)
- moved U4 1.52 mm to (127.0, 71.4)
- moved R53 0.25 mm to (101.6, 110.7)
Routing:
- net /AGND: track 0.00 -> 797.3 mm
- net /GND: track 50.6 -> 789.9 mm, vias 0 -> 2
- net /3V3_TNY: track 0.00 -> 348.4 mm, vias 0 -> 6
- net /DIR0: track 0.00 -> 291.2 mm
- net /+12V: track 0.00 -> 278.2 mm
- net /HW_EN: track 0.00 -> 275.6 mm
- net /10V_REF: track 0.00 -> 270.7 mm, vias 0 -> 5
- net /CLK1: track 0.00 -> 250.7 mm
- net /-12V: track 0.00 -> 248.6 mm
- net /CLK0: track 0.00 -> 235.6 mm
- net /DIR1: track 0.00 -> 228.3 mm, vias 0 -> 2
- net /SG9: track 0.00 -> 227.3 mm
- net N-0000035: track 0.00 -> 224.7 mm
- net /SG8: track 0.00 -> 208.2 mm
- net /DIR4: track 0.00 -> 206.5 mm, vias 0 -> 1
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Other:
- board text added: "+"
- board text added: "-"
- board text added: "5V_SEL"
- board text added: "AOUT"
- board text added: "CAMERA TRIGGERS"
- board text added: "CLK3"
- board text added: "CLK4"
- board text added: "D0"
- board text added: "D1"
- board text added: "DIGITAL OUTPUTS"
- board text added: "DIR3"
- board text added: "DIR4"
- board text added: "EXT"
- board text added: "HOMING SWITCHES"
- board text added: "INT0"
- board text added: "LIMIT/KILL SWITCHES"
- board text added: "MIRROR DIR0 POLARITY"
- board text added: "MIRROR DIR1 POLARITY"
- board text added: "MIRRORED MOTOR OUTPUTS"
- board text added: "MOTOR 3"
- board text added: "MOTOR 4"
- board text added: "MOTOR OUTPUTS"
- board text added: "NOAH WATER TUNNEL MOTION CONTROLLER V0.1 R1 www.iorodeo.com"
- board text added: "OPTIONAL 5V EXT PWR"
- board text added: "OPTIONAL F/T 5V PWR"
- board text added: "PWM/RC-SERVO"
- board text added: "PWM0"
- board text added: "PWM1"
- board text added: "PWM2"
- board text added: "PWM3"
- board text added: "PWM4"
- board text added: "SWITCH0"
- board text added: "SWITCH1"
- board text added: "SWITCH2"
- board text added: "TNY"
- board text added: "TRIG0"
- board text added: "TRIG1"
- board text added: "UEXT"
